Commit message: adds tf broadcasts to sensors_node, includes miniboat geometry in rviz, moves visualization to roboat_visualization new package

File: roboat_localization/urdf/roboat.urdf.xacro (robot description, xacro)
@@ -24,5 +24,5 @@
             <origin xyz="0 0 0.0"/>
             <geometry>
-                <mesh filename="package://roboat_localization/meshes/roboat.dae" />
+                <mesh filename="package://roboat_visualization/meshes/miniboat.dae" />
             </geometry>
         </collision>
@@ -30,5 +30,5 @@
             <origin xyz="0 0 0.0"/>
             <geometry>
-                <mesh filename="package://roboat_localization/meshes/roboat.dae" />
+                <mesh filename="package://roboat_visualization/meshes/miniboat.dae" />
             </geometry>
         </visual>

Commit message: moves roboat_visualizaton node to server, enables multiple base_link frames

File: roboat_localization/urdf/roboat.urdf.xacro (robot description, xacro)
@@ -1,4 +1,8 @@
 <?xml version="1.0"?>
-<robot name="roboat" xmlns:xacro="http://roboat.org">
+<robot name="miniboat" xmlns:xacro="http://roboat.org">
+    <!-- arguments -->
+    <xacro:arg name="id" default="miniboat" />
+    <!-- constants -->
+    <xacro:property name="id" value="$(arg id)" />
     <xacro:property name="PI" value="3.1415926535897931"/>
     <material name="dark_grey">
@@ -14,11 +18,11 @@
         <color rgba="0.15 0.15 0.15 1.0"/>
     </material>
-    <link name="base_link"/>
-    <joint name="base_link_joint" type="fixed">
-        <parent link="base_link"/>
-        <child link="chassis_link"/>
+    <link name="base_link_${id}"/>
+    <joint name="base_link_joint_${id}" type="fixed">
+        <parent link="base_link_${id}"/>
+        <child link="chassis_link_${id}"/>
         <origin xyz="0 0 0.5" rpy="0 0 0"/>
     </joint>
-    <link name="chassis_link">
+    <link name="chassis_link_${id}">
         <collision>
             <origin xyz="0 0 0.0"/>
@@ -44,20 +48,20 @@
         </inertial>
     </link>
-    <link name="imu_link"/>
-    <joint name="imu_joint" type="fixed">
-        <parent link="chassis_link"/>
-        <child link="imu_link"/>
+    <link name="imu_link_${id}"/>
+    <joint name="imu_joint_${id}" type="fixed">
+        <parent link="chassis_link_${id}"/>
+        <child link="imu_link_${id}"/>
         <origin xyz="1.8 0 1.2" rpy="0 0 0"/>
     </joint>
-    <link name="navsat_link"/>
-    <joint name="navsat_joint" type="fixed">
-        <parent link="chassis_link"/>
-        <child link="navsat_link"/>
+    <link name="navsat_link_${id}"/>
+    <joint name="navsat_joint_${id}" type="fixed">
+        <parent link="chassis_link_${id}"/>
+        <child link="navsat_link_${id}"/>
         <origin xyz="1.8 -0.45 1.2" rpy="0 0 0"/>
     </joint>
-    <link name="navsat2_link"/>
-    <joint name="navsat2_joint" type="fixed">
-        <parent link="chassis_link"/>
-        <child link="navsat2_link"/>
+    <link name="navsat2_link_${id}"/>
+    <joint name="navsat2_joint_${id}" type="fixed">
+        <parent link="chassis_link_${id}"/>
+        <child link="navsat2_link_${id}"/>
         <origin xyz="-1.8 0.45 1.2" rpy="0 0 0"/>
     </joint>

Commit message: moves sensor_node to roboat_localization

File: roboat_localization/urdf/roboat.urdf.xacro (robot description, xacro)
@@ -18,11 +18,5 @@
         <color rgba="0.15 0.15 0.15 1.0"/>
     </material>
-    <link name="base_link_${id}"/>
-    <joint name="base_link_joint_${id}" type="fixed">
-        <parent link="base_link_${id}"/>
-        <child link="chassis_link_${id}"/>
-        <origin xyz="0 0 0.5" rpy="0 0 0"/>
-    </joint>
-    <link name="chassis_link_${id}">
+    <link name="base_link_${id}">
         <collision>
             <origin xyz="0 0 0.0"/>
@@ -39,30 +33,30 @@
         <inertial>
             <!-- Center of mass -->
-            <origin xyz="0 0 0.7" rpy="0 0 0"/>
-            <mass value="1300.523"/>
-            <!-- Moments of inertia: ( chassis without wheels ) -->
+            <origin xyz="0 0 0.05" rpy="0 0 0"/>
+            <mass value="0.6"/>
+            <!-- Moments of inertia -->
             <inertia
-                    ixx="10.3136" ixy="-10.0008" ixz="10.0164"
-                    iyy="10.3922" iyz="-10.0009"
-                    izz="10.4485"/>
+                    ixx="0.009" ixy="0.0" ixz="0.0"
+                    iyy="0.009" iyz="0.0"
+                    izz="0.006"/>
         </inertial>
     </link>
     <link name="imu_link_${id}"/>
     <joint name="imu_joint_${id}" type="fixed">
-        <parent link="chassis_link_${id}"/>
+        <parent link="base_link_${id}"/>
         <child link="imu_link_${id}"/>
-        <origin xyz="1.8 0 1.2" rpy="0 0 0"/>
+        <origin xyz="0.0 0.0 0.04" rpy="0 0 0"/>
     </joint>
-    <link name="navsat_link_${id}"/>
-    <joint name="navsat_joint_${id}" type="fixed">
-        <parent link="chassis_link_${id}"/>
-        <child link="navsat_link_${id}"/>
-        <origin xyz="1.8 -0.45 1.2" rpy="0 0 0"/>
+    <link name="beacon1_link_${id}"/>
+    <joint name="beacon1_joint_${id}" type="fixed">
+        <parent link="base_link_${id}"/>
+        <child link="beacon1_link_${id}"/>
+        <origin xyz="0.09 0.09 0.09" rpy="0 0 0"/>
     </joint>
-    <link name="navsat2_link_${id}"/>
-    <joint name="navsat2_joint_${id}" type="fixed">
-        <parent link="chassis_link_${id}"/>
-        <child link="navsat2_link_${id}"/>
-        <origin xyz="-1.8 0.45 1.2" rpy="0 0 0"/>
+    <link name="beacon2_link_${id}"/>
+    <joint name="beacon2_joint_${id}" type="fixed">
+        <parent link="base_link_${id}"/>
+        <child link="beacon2_link_${id}"/>
+        <origin xyz="-0.09 -0.09 0.09" rpy="0 0 0"/>
     </joint>
 </robot>

Commit message: changes "state" to "odom/filtered" topic to align with EKF notation

File: roboat_localization/urdf/roboat.urdf.xacro (robot description, xacro)
@@ -18,5 +18,7 @@
         <color rgba="0.15 0.15 0.15 1.0"/>
     </material>
-    <link name="base_link_${id}">
+    <link name="base_link_${id}"/>
+    <!-- KDL does not support a base_link with an inertia. As workaround, we add an extra dummy link -->
+    <link name="chassis_link_${id}">
         <collision>
             <origin xyz="0 0 0.0"/>
@@ -42,4 +44,10 @@
         </inertial>
     </link>
+    <joint name="chassis_joint_${id}" type="fixed">
+        <parent link="base_link_${id}"/>
+        <child link="chassis_link_${id}"/>
+        <origin xyz="0 0 0" rpy="0 0 0"/>
+    </joint>
+    <!-- sensor joints -->
     <link name="imu_link_${id}"/>
     <joint name="imu_joint_${id}" type="fixed">

Commit message: enables EKF in roboat_localization

File: roboat_localization/urdf/roboat.urdf.xacro (robot description, xacro)
@@ -18,4 +18,5 @@
         <color rgba="0.15 0.15 0.15 1.0"/>
     </material>
+    <!-- miniboat root link -->
     <link name="base_link_${id}"/>
     <!-- KDL does not support a base_link with an inertia. As workaround, we add an extra dummy link -->
@@ -56,15 +57,9 @@
         <origin xyz="0.0 0.0 0.04" rpy="0 0 0"/>
     </joint>
-    <link name="beacon1_link_${id}"/>
+    <link name="dual_beacon_link_${id}"/>
     <joint name="beacon1_joint_${id}" type="fixed">
         <parent link="base_link_${id}"/>
-        <child link="beacon1_link_${id}"/>
-        <origin xyz="0.09 0.09 0.09" rpy="0 0 0"/>
-    </joint>
-    <link name="beacon2_link_${id}"/>
-    <joint name="beacon2_joint_${id}" type="fixed">
-        <parent link="base_link_${id}"/>
-        <child link="beacon2_link_${id}"/>
-        <origin xyz="-0.09 -0.09 0.09" rpy="0 0 0"/>
+        <child link="dual_beacon_link_${id}"/>
+        <origin xyz="0.0 0.0 0.09" rpy="0 0 ${135*PI/180.0}"/>
     </joint>
 </robot>

Commit message: adjusts paths in install/update scripts

File: roboat_localization/urdf/roboat.urdf.xacro (robot description, xacro)
@@ -58,5 +58,5 @@
     </joint>
     <link name="dual_beacon_link_${id}"/>
-    <joint name="beacon1_joint_${id}" type="fixed">
+    <joint name="dual_beacon_joint_${id}" type="fixed">
         <parent link="base_link_${id}"/>
         <child link="dual_beacon_link_${id}"/>
